Commit message: fix robot description

File: rover_ws/src/rover_description/urdf/camera.xacro (robot description, xacro)
@@ -1,11 +1,9 @@
 <?xml version="1.0"?>
 <robot xmlns:xacro="http://www.ros.org/wiki/xacro">
-<!-- camera.xacro -->
-<joint name="camera_joint" type="fixed">
-  <parent link="chassis"/>
-  <child link="camera_link"/>
-  <origin xyz="0.335 -0.001 0.09" rpy="0 -0.611 0"/>
-  <!--                                    ↑ -35° in radians -->
-</joint>
+    <joint name="camera_joint" type="fixed">
+        <parent link="chassis"/>
+        <child link="camera_link"/>
+        <origin xyz="0.335 -0.001 0.09" rpy="0 0 0"/>
+    </joint>
     <link name="camera_link">
         <visual>

File: rover_ws/src/rover_description/urdf/gazebo_control.xacro (robot description, xacro)
@@ -4,5 +4,4 @@
         <!-- <plugin name="diff_drive" filename="libgazebo_ros_diff_drive.so"> -->
         <plugin filename="gz-sim-diff-drive-system" name="gz::sim::systems::DiffDrive">
-            <topic>cmd_vel</topic>
             <!-- Wheel Information -->
             <left_joint>left_wheel_joint</left_joint>

File: rover_ws/src/rover_description/urdf/ros2_control.xacro (robot description, xacro)
@@ -18,6 +18,6 @@
                     <param name="max">10</param>
                 </command_interface>
+                <state_interface name="velocity"/>
                 <state_interface name="position"/>
-                <state_interface name="velocity"/>
             </joint>
             <joint name="right_wheel_joint">
@@ -26,6 +26,6 @@
                     <param name="max">10</param>
                 </command_interface>
+                <state_interface name="velocity"/>
                 <state_interface name="position"/>
-                <state_interface name="velocity"/>
             </joint>
         </ros2_control>
@@ -61,6 +61,6 @@
         </plugin>
     </gazebo> -->
-<gazebo>
-  <plugin filename="libgz_ros2_control-system.so" name="gz_ros2_control::GazeboSimROS2ControlPlugin">
+    <gazebo>
+  <plugin filename="gz_ros2_control-system" name="gz_ros2_control::GazeboSimROS2ControlPlugin">
     <parameters>$(find rover_controller)/config/my_controllers.yaml</parameters>
     <parameters>$(find rover_description)/config/gaz_ros2_ctl_use_sim.yaml</parameters>

File: rover_ws/src/rover_description/urdf/rover_core.xacro (robot description, xacro)
@@ -16,5 +16,4 @@
     <xacro:property name="caster_wheel_offset_x" value="0.075"/>
     <xacro:property name="caster_wheel_offset_z" value="${wheel_offset_z - wheel_radius + caster_wheel_radius}"/>
-    <xacro:property name="mast_radius" value="0.015"/> <xacro:property name="mast_height" value="0.028"/>  ```
     <material name="rover_white">
         <color rgba="1 1 1 1" />
@@ -119,5 +118,5 @@
         <collision>
             <geometry>
-                <sphere radius="${wheel_radius}" length="${wheel_thickness}"/>
+               <cylinder radius="${wheel_radius}" length="${wheel_thickness}"/>
             </geometry>
         </collision>

Commit message: few modifications

File: rover_ws/src/rover_description/urdf/camera.xacro (robot description, xacro)
@@ -1,8 +1,9 @@
 <?xml version="1.0"?>
 <robot xmlns:xacro="http://www.ros.org/wiki/xacro">
+    <xacro:property name="camera_tilt" value="0.0"/>  <!-- radians, positive = tilt down -->
     <joint name="camera_joint" type="fixed">
-        <parent link="chassis"/>
-        <child link="camera_link"/>
-        <origin xyz="0.335 -0.001 0.09" rpy="0 0 0"/>
+    <parent link="chassis"/>
+    <child link="camera_link"/>
+    <origin xyz="0.335 -0.001 0.09" rpy="0 ${camera_tilt} 0"/>
     </joint>
     <link name="camera_link">

Commit message: pitch change allowble in simulation

File: rover_ws/src/rover_description/urdf/camera.xacro (robot description, xacro)
@@ -1,9 +1,11 @@
 <?xml version="1.0"?>
 <robot xmlns:xacro="http://www.ros.org/wiki/xacro">
-    <xacro:property name="camera_tilt" value="0.0"/>  <!-- radians, positive = tilt down -->
+    <!-- 1. Keep your tilt property here -->
+    <xacro:property name="camera_tilt" value="${15 * pi / 180}"/>
+    <!-- 2. Keep the physical housing straight relative to the chassis -->
     <joint name="camera_joint" type="fixed">
-    <parent link="chassis"/>
-    <child link="camera_link"/>
-    <origin xyz="0.335 -0.001 0.09" rpy="0 ${camera_tilt} 0"/>
+        <parent link="chassis"/>
+        <child link="camera_link"/>
+        <origin xyz="0.335 -0.001 0.09" rpy="0 0 0"/>
     </joint>
     <link name="camera_link">
@@ -15,17 +17,14 @@
             <material name="rover_red"/>
         </visual>
-        <!-- <collision>
-            <origin xyz="0 0 0" rpy="0 0 0"/>
-            <geometry>
-                <box size="0.010 0.03 0.03"/>
-            </geometry>
-        </collision> -->
     </link>
+    <!-- 3. Inject the camera tilt directly into the optical transform chain -->
+    <!-- Default optical is rpy="${-pi/2} 0 ${-pi/2}". We add the tilt into the Pitch (middle value) -->
     <joint name="camera_optical_joint" type="fixed">
         <parent link="camera_link"/>
         <child link="camera_link_optical"/>
-        <origin xyz="0 0 0" rpy="${-pi/2} 0 ${-pi/2}"/>
+        <origin xyz="0 0 0" rpy="${-pi/2} ${camera_tilt} ${-pi/2}" />
     </joint>
     <link name="camera_link_optical"></link>
+    <!-- 4. Revert Gazebo back to tracking the un-tilted base link -->
     <gazebo reference="camera_link">
         <sensor name="camera" type="rgbd_camera">

Commit message: correct tilting

File: rover_ws/src/rover_description/urdf/camera.xacro (robot description, xacro)
@@ -1,31 +1,29 @@
 <?xml version="1.0"?>
 <robot xmlns:xacro="http://www.ros.org/wiki/xacro">
-    <xacro:property name="camera_tilt" value="0.0"/>  <!-- radians, positive = tilt down -->
+    <!-- 1. Define your camera tilt (e.g., 15 degrees down) -->
+    <xacro:property name="camera_tilt" value="${15 * pi / 180}" />
+    <!-- 2. Apply the physical tilt HERE. This tilts both the physical box and the sensor -->
     <joint name="camera_joint" type="fixed">
-    <parent link="chassis"/>
-    <child link="camera_link"/>
-    <origin xyz="0.335 -0.001 0.09" rpy="0 ${camera_tilt} 0"/>
+        <parent link="chassis" />
+        <child link="camera_link" />
+        <origin xyz="0.335 -0.001 0.09" rpy="0 ${camera_tilt} 0" />
     </joint>
     <link name="camera_link">
         <visual>
-            <origin xyz="0 0 0" rpy="0 0 0"/>
+            <origin xyz="0 0 0" rpy="0 ${camera_tilt} 0" />
             <geometry>
-                <box size="0.010 0.03 0.03"/>
+                <box size="0.010 0.03 0.03" />
             </geometry>
-            <material name="rover_red"/>
+            <material name="rover_red" />
         </visual>
-        <!-- <collision>
-            <origin xyz="0 0 0" rpy="0 0 0"/>
-            <geometry>
-                <box size="0.010 0.03 0.03"/>
-            </geometry>
-        </collision> -->
     </link>
+    <!-- 3. Return the optical joint to its standard, static ROS rotation -->
     <joint name="camera_optical_joint" type="fixed">
-        <parent link="camera_link"/>
-        <child link="camera_link_optical"/>
-        <origin xyz="0 0 0" rpy="${-pi/2} 0 ${-pi/2}"/>
+        <parent link="camera_link" />
+        <child link="camera_link_optical" />
+        <origin xyz="0 0 0" rpy="${-pi/2} 0 ${-pi/2}" />
     </joint>
     <link name="camera_link_optical"></link>
+    <!-- 4. Gazebo Sensor Configuration -->
     <gazebo reference="camera_link">
         <sensor name="camera" type="rgbd_camera">
@@ -33,4 +31,5 @@
             <update_rate>30</update_rate>
             <topic>camera</topic>
+            <!-- Use camera_link so Gazebo tilts the camera sensor frame naturally -->
             <gz_frame_id>camera_link</gz_frame_id>
             <camera name="camera">

Commit message: lane following

File: rover_ws/src/rover_description/urdf/camera.xacro (robot description, xacro)
@@ -2,10 +2,10 @@
 <robot xmlns:xacro="http://www.ros.org/wiki/xacro">
     <!-- 1. Keep your tilt property here -->
-    <xacro:property name="camera_tilt" value="${15 * pi / 180}"/>
+    <xacro:property name="camera_tilt" value="${0 * pi / 180}"/>
     <!-- 2. Keep the physical housing straight relative to the chassis -->
     <joint name="camera_joint" type="fixed">
         <parent link="chassis"/>
         <child link="camera_link"/>
-        <origin xyz="0.335 -0.001 0.09" rpy="0 0 0"/>
+        <origin xyz="0.335 -0.001 0.1" rpy="0 ${camera_tilt} 0"/>
     </joint>
     <link name="camera_link">
@@ -23,5 +23,5 @@
         <parent link="camera_link"/>
         <child link="camera_link_optical"/>
-        <origin xyz="0 0 0" rpy="${-pi/2} ${camera_tilt} ${-pi/2}" />
+        <origin xyz="0 0 0" rpy="${-pi/2} 0 ${-pi/2}" />
     </joint>
     <link name="camera_link_optical"></link>
@@ -42,10 +42,10 @@
                 <clip>
                     <near>0.01</near>
-                    <far>10.0</far>
+                    <far>90.0</far>
                 </clip>
                 <depth_camera>
                     <clip>
                         <near>0.1</near>
-                        <far>10.0</far>
+                        <far>90.0</far>
                     </clip>
                 </depth_camera>
